File: ORION_sub_v2.kicad_sch (KiCad schematic)
At the start: 75 parts, among them J1 Conn_01x02, J10 Conn_01x01, J11 Conn_01x05, J12 Conn_01x03, J13 Conn_01x08, J2 Conn_01x03, J3 Conn_01x04, J4 Conn_01x02, J5 Conn_01x01, J6 Conn_01x04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

Commit message: 更新
Parts:
- added D8: D_Zener, Diode_SMD:D_0805_2012Metric, symbol Device:D_Zener
- added Q2: Q_PMOS_GDS, Package_TO_SOT_SMD:TO-252-2, symbol Device:Q_PMOS_GDS
- added Q3: BSS138, Package_TO_SOT_SMD:SOT-23, symbol Transistor_FET:BSS138
- added R28, R29, R30: 1k, Resistor_SMD:R_0603_1608Metric, symbol SSL_BST_ver1.3-rescue:R
- R2: value 120 -> 1k
Connections:
- net +BATT: now also D8.1 (K), Q2.3 (S), R29.1
- net GND: now also Q3.2 (S), R30.2
- new net: D8.2 (A), Q2.1 (G), R28.1, R29.2
- new net: Q3.3 (D), R28.2
- new net ESC_BATT: Q2.2 (D)
- new net ESC_BATT_EN: Q3.1 (G), R30.1
Other:
- moved on the sheet: C12, C13, C3, C4, C7, C8, D1, D10, D2, D3, D4, D5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
